File: compact-photodiode-v2/compact_photodiode_v2.kicad_pcb (KiCad board)
At the start: 2 copper layers, 34.4 x 18 mm, 3 parts, among them U1 OPT101P

Commit message: do something
Parts:
- moved U2 7.61 mm to (149.0, 122.5)
Changed lines of the file:
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@@
 			(psa4output no)
 			(plot_black_and_white yes)
-			(plotinvisibletext no)
 			(sketchpadsonfab no)
 			(plotpadnumbers no)
@@
 	(footprint "RF_Connectors_Footprints:SMB_Molex_0731000103_THT_RA"
 		(layer "F.Cu")
-		(at 148.6 114.9 180)
+		(at 149 122.5 180)
 		(property "Reference" "U2"
 			(at 0 -17 180)

Commit message: add library
Parts:
- moved U2 0.97 mm to (148.1, 122.7)
Routing:
- net GND: track 50.3 -> 65.1 mm
- net Net-(U1-FB): track 35.2 -> 32.5 mm
Changed lines of the file:
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@@
 			(psa4output no)
 			(plot_black_and_white yes)
+			(plotinvisibletext no)
 			(sketchpadsonfab no)
 			(plotpadnumbers no)
@@
 	(footprint "RF_Connectors_Footprints:SMB_Molex_0731000103_THT_RA"
 		(layer "F.Cu")
-		(at 149 122.5 180)
+		(at 148.06 122.74 180)
 		(property "Reference" "U2"
 			(at 0 -17 180)
@@
 		(fp_line
 			(start 4 -4)
-			(end 2.5 -4.5)
-			(stroke
-				(width 0.05)
-				(type default)
-			)
-			(layer "F.CrtYd")
-		)
-		(fp_line
-			(start 2.5 -4.5)
-			(end 2.5 -11)
-			(stroke
-				(width 0.05)
-				(type default)
-			)
-			(layer "F.CrtYd")
-		)
-		(fp_line
-			(start 2.5 -11)
-			(end -2.5 -11)
-			(stroke
-				(width 0.05)
-				(type default)
-			)
-			(layer "F.CrtYd")
-		)
-		(fp_line
-			(start -2.5 -4.5)
 			(end -4 -4)
-			(stroke
-				(width 0.05)
-				(type default)
-			)
-			(layer "F.CrtYd")
-		)
-		(fp_line
-			(start -2.5 -11)
-			(end -2.5 -4.5)
 			(stroke
 				(width 0.05)
@@
 		)
 		(pad "1" thru_hole rect
-			(at -2.54 2.54 270)
+			(at -2.54 -2.54 270)
 			(size 2.7 2.7)
 			(drill 1.7)
@@
 		)
 		(pad "1" thru_hole rect
-			(at -2.397825 -2.586554 270)
+			(at -2.54 2.54 270)
 			(size 2.7 2.7)
 			(drill 1.7)
@@
 	)
 	(segment
-		(start 146.06 112.36)
-		(end 146.06 117.44)
+		(start 137.45 117.8)
+		(end 135.824 116.174)
 		(width 0.25)
 		(layer "F.Cu")
@@
 	)
 	(segment
-		(start 146.06 117.44)
-		(end 146.16 117.44)
+		(start 145.52 120.2)
+		(end 145.52 125.28)
 		(width 0.25)
 		(layer "F.Cu")
@@
 	)
 	(segment
-		(start 143.874 110.174)
-		(end 146.06 112.36)
+		(start 150.6 125.28)
+		(end 144.93 125.28)
 		(width 0.25)
 		(layer "F.Cu")
@@
 	)
 	(segment
-		(start 146.06 112.36)
-		(end 151.23 112.36)
+		(start 149.044 110.174)
+		(end 155.39 116.52)
 		(width 0.25)
 		(layer "F.Cu")
@@
 	)
 	(segment
-		(start 146.16 117.44)
-		(end 146.206554 117.486554)
+		(start 135.824 116.174)
+		(end 135.824 110.174)
+		(width 0.25)
+		(layer "F.Cu")
+		(net 1)
+	)
+	(segment
+		(start 135.824 110.174)
+		(end 149.044 110.174)
+		(width 0.25)
+		(layer "F.Cu")
+		(net 1)
+	)
+	(segment
+		(start 139.85 120.2)
+		(end 137.45 117.8)
+		(width 0.25)
+		(layer "F.Cu")
+		(net 1)
+	)
+	(segment
+		(start 145.52 120.2)
+		(end 139.85 120.2)
+		(width 0.25)
+		(layer "F.Cu")
+		(net 1)
+	)
+	(segment
+		(start 150.6 120.2)
+		(end 145.52 120.2)
 		(width 0.25)
 		(layer "F.Cu")
@@
 	)
 	(segment
-		(start 146.206554 117.486554)
-		(end 150.997825 117.486554)
-		(width 0.25)
-		(layer "F.Cu")
-		(net 1)
-	)
-	(segment
-		(start 135.824 116.174)
-		(end 135.824 110.174)
-		(width 0.25)
-		(layer "F.Cu")
-		(net 1)
-	)
-	(segment
-		(start 151.23 112.36)
-		(end 155.39 116.52)
-		(width 0.25)
-		(layer "F.Cu")
-		(net 1)
-	)
-	(segment
-		(start 137.45 117.8)
-		(end 135.824 116.174)
-		(width 0.25)
-		(layer "F.Cu")
-		(net 1)
-	)
-	(segment
-		(start 135.824 110.174)
-		(end 143.874 110.174)
-		(width 0.25)
-		(layer "F.Cu")
-		(net 1)
-	)
-	(segment
 		(start 155.39 116.52)
 		(end 157.93 116.52)
@@
 	)
 	(segment
+		(start 155.39 121.39)
+		(end 155.39 121.6)
+		(width 0.25)
+		(layer "F.Cu")
+		(net 2)
+	)
+	(segment
+		(start 137.45 111.8)
+		(end 145.8 111.8)
+		(width 0.25)
+		(layer "F.Cu")
+		(net 2)
+	)
+	(segment
+		(start 145.8 111.8)
+		(end 155.39 121.39)
+		(width 0.25)
+		(layer "F.Cu")
+		(net 2)
+	)
+	(segment
 		(start 137.45 111.8)
 		(end 137.45 112.45)
@@
 	)
 	(segment
-		(start 146.6 121.6)
-		(end 155.39 121.6)
-		(width 0.25)
-		(layer "F.Cu")
-		(net 2)
-	)
-	(segment
-		(start 137.45 112.45)
-		(end 146.6 121.6)
-		(width 0.25)
-		(layer "F.Cu")
-		(net 2)
-	)
-	(segment
-		(start 163.476405 122.726)
-		(end 164.136 122.066405)
+		(start 164.136 122.066405)
+		(end 164.136 115.106)
 		(width 0.25)
 		(layer "F.Cu")
@@
 	)
 	(segment
-		(start 157.463595 117.646)
-		(end 162.543595 122.726)
+		(start 148.06 122.74)
+		(end 163.462405 122.74)
 		(width 0.25)
 		(layer "F.Cu")
@@
 	)
 	(segment
-		(start 162.543595 122.726)
-		(end 163.476405 122.726)
+		(start 155.39 113.98)
+		(end 163.01 113.98)
 		(width 0.25)
 		(layer "F.Cu")
@@
 	)
 	(segment
-		(start 154.646 117.646)
-		(end 157.463595 117.646)
-		(width 0.25)
-		(layer "F.Cu")
-		(net 4)
-	)
-	(segment
-		(start 151.9 114.9)
-		(end 154.646 117.646)
-		(width 0.25)
-		(layer "F.Cu")
-		(net 4)
-	)
-	(segment
-		(start 148.6 114.9)
-		(end 151.9 114.9)
-		(width 0.25)
-		(layer "F.Cu")
-		(net 4)
-	)
-	(segment
-		(start 164.136 122.066405)
-		(end 164.136 115.106)
-		(width 0.25)
-		(layer "F.Cu")
-		(net 4)
-	)
-	(segment
-		(start 163.01 113.98)
-		(end 155.39 113.98)
-		(width 0.25)
-		(layer "F.Cu")
+		(start 163.462405 122.74)
+		(end 164.136 122.066405)
+		(width 0.25)
+		(layer "F.Cu")
