File: compact-photodiode-v2/compact_photodiode_v2.kicad_pcb (KiCad board)
At the start: 2 copper layers, 34.4 x 18 mm, 3 parts, among them U1 OPT101P

Commit message: Add text
Other:
- board text added: "Designed by Olgierd Matusiewicz"

Commit message: Do something
Parts:
- added C1: C, Capacitor_SMD:C_0603_1608Metric_Pad1.08x0.95mm_HandSolder, B.Cu at (148.4, 115.5)
- added R2: CF14JT5M10, footprints:STA_CF14_STP, F.Cu at (143.6, 111.5)
Connections:
- U1 pad 2: unconnected-(U1--IN-Pad2) -> Net-(U1--IN)
- U1 pad 4: Net-(U1-FB) -> unconnected-(U1-FB-Pad4)
- U1 pad 5: Net-(U1-FB) -> Net-(U1-OUT)
- U2 pad 2: Net-(U1-FB) -> Net-(U1-OUT)
Routing:
- net Net-(U1-FB): track 32.5 -> 0.00 mm
- net Net-(U1-OUT): track 0.00 -> 26.6 mm
- net Net-(U1--IN): track 0.00 -> 24.8 mm
- net GND: track 65.1 -> 48.6 mm
Other:
- board text added: "1MΩ=3pF"
- board text added: "WayWayWay"

Commit message: Start MCU Project
Parts:
- renumbered U2 to BNC, R2 to R1
Other:
- board text added: "CH33-SE"
- board text removed: "WayWayWay"
Changed lines of the file:
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@@
 		(at 143.57 111.5)
 		(tags "CF14JT5M10 ")
-		(property "Reference" "R2"
+		(property "Reference" "R1"
 			(at 5.715 0 0)
 			(unlocked yes)
@@
 		(layer "F.Cu")
 		(at 148.06 122.74 180)
-		(property "Reference" "U2"
+		(property "Reference" "BNC"
 			(at -4.94 -0.76 90)
 			(unlocked yes)
@@
 		)
 	)
-	(gr_text "WayWayWay"
+	(gr_text "CH33-SE"
 		(at 155 126.5 0)
 		(layer "F.SilkS")
