File: compact-photodiode-v2/compact_photodiode_v2.kicad_sch (KiCad schematic)
At the start: 3 parts, among them U1 OPT101P

Commit message: add library
Parts:
- U2: footprint RF_Connectors_Footprints:SMB_Molex_0731000103_THT_RA -> 0731000103:SMB_Molex_0731000103_THT_RA
Changed lines of the file:
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@@
 			)
 		)
-		(property "Footprint" "RF_Connectors_Footprints:SMB_Molex_0731000103_THT_RA"
+		(property "Footprint" "0731000103:SMB_Molex_0731000103_THT_RA"
 			(at 153.67 124.46 0)
 			(effects

Commit message: Do something
Parts:
- added C1: C, Capacitor_SMD:C_0603_1608Metric_Pad1.08x0.95mm_HandSolder, symbol Device:C
- added R2: CF14JT5M10, footprints:STA_CF14_STP, symbol 2025-06-12_23-46-23:CF14JT5M10
Connections:
- net at U1.2 (-IN): now also C1.2, R2.1
- net at U1.5 (OUT), U2.2 (IN): now also C1.1, R2.2; no longer U1.4 (FB)
Changed lines of the file:
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@@
+	)
+	(junction
+		(at 135.89 106.68)
+		(diameter 0)
+		(color 0 0 0 0)
+	)
+	(junction
+		(at 135.89 99.06)
+		(diameter 0)
+		(color 0 0 0 0)
 	)
 	(junction
@@
 	)
 	(no_connect
-		(at 138.43 106.68)
+		(at 138.43 109.22)
 	)
 	(wire
@@
 	(wire
 		(pts
-			(xy 134.62 97.79) (xy 157.48 97.79)
-		)
-		(stroke
-			(width 0)
-			(type default)
-		)
-	)
-	(wire
-		(pts
-			(xy 138.43 109.22) (xy 134.62 109.22)
+			(xy 135.89 106.68) (xy 138.43 106.68)
+		)
+		(stroke
+			(width 0)
+			(type default)
+		)
+	)
+	(wire
+		(pts
+			(xy 134.62 99.06) (xy 135.89 99.06)
 		)
 		(stroke
@@
 	(wire
 		(pts
-			(xy 134.62 109.22) (xy 134.62 97.79)
-		)
-		(stroke
-			(width 0)
-			(type default)
-		)
-	)
-	(wire
-		(pts
 			(xy 189.23 101.6) (xy 177.8 101.6)
 		)
@@
 	(wire
 		(pts
-			(xy 157.48 97.79) (xy 157.48 109.22)
+			(xy 157.48 99.06) (xy 157.48 109.22)
+		)
+		(stroke
+			(width 0)
+			(type default)
+		)
+	)
+	(wire
+		(pts
+			(xy 135.89 99.06) (xy 157.48 99.06)
+		)
+		(stroke
+			(width 0)
+			(type default)
+		)
+	)
+	(wire
+		(pts
+			(xy 121.92 106.68) (xy 135.89 106.68)
 		)
 		(stroke
@@
 		(pts
 			(xy 153.67 109.22) (xy 153.67 118.11)
+		)
+		(stroke
+			(width 0)
+			(type default)
+		)
+	)
+	(wire
+		(pts
+			(xy 121.92 106.68) (xy 121.92 99.06)
 		)
 		(stroke
@@
 	)
 	(symbol
+		(lib_id "2025-06-12_23-46-23:CF14JT5M10")
+		(at 121.92 99.06 0)
+		(unit 1)
+		(exclude_from_sim no)
+		(in_bom yes)
+		(on_board yes)
+		(dnp no)
+		(fields_autoplaced yes)
+		(property "Reference" "R2"
+			(at 128.27 92.71 0)
+			(effects
+				(font
+					(size 1.524 1.524)
+				)
+			)
+		)
+		(property "Value" "CF14JT5M10"
+			(at 128.27 95.25 0)
+			(effects
+				(font
+					(size 1.524 1.524)
+				)
+			)
+		)
+		(property "Footprint" "footprints:STA_CF14_STP"
+			(at 121.92 99.06 0)
+			(effects
+				(font
+					(size 1.27 1.27)
+					(italic yes)
+				)
+				(hide yes)
+			)
+		)
+		(property "Datasheet" "CF14JT5M10"
+			(at 121.92 99.06 0)
+			(effects
+				(font
+					(size 1.27 1.27)
+					(italic yes)
+				)
+				(hide yes)
+			)
+		)
+		(property "Description" ""
+			(at 121.92 99.06 0)
+			(effects
+				(font
+					(size 1.27 1.27)
+				)
+				(hide yes)
+			)
+		)
+		(pin "2"
+		)
+		(pin "1"
+		)
+		(instances
+			(project ""
+				(path "/cfa4a98a-fd35-4db5-8ff8-6d1775bad148"
+					(reference "R2")
+					(unit 1)
+				)
+			)
+		)
+	)
+	(symbol
 		(lib_id "power:PWR_FLAG")
 		(at 177.8 101.6 0)
@@
 					(unit 1)
 				)
+			)
+		)
+	)
+	(symbol
+		(lib_id "Device:C")
+		(at 135.89 102.87 0)
+		(unit 1)
+		(exclude_from_sim no)
+		(in_bom yes)
+		(on_board yes)
+		(dnp no)
+		(fields_autoplaced yes)
+		(property "Reference" "C1"
+			(at 139.7 101.5999 0)
+			(effects
+				(font
+					(size 1.27 1.27)
+				)
+				(justify left)
+			)
+		)
+		(property "Value" "C"
+			(at 139.7 104.1399 0)
+			(effects
+				(font
+					(size 1.27 1.27)
+				)
+				(justify left)
+			)
+		)
+		(property "Footprint" "Capacitor_SMD:C_0603_1608Metric_Pad1.08x0.95mm_HandSolder"
+			(at 136.8552 106.68 0)
+			(effects
+				(font
+					(size 1.27 1.27)
+				)
+				(hide yes)
+			)
+		)
+		(property "Datasheet" "~"
+			(at 135.89 102.87 0)
+			(effects
+				(font
+					(size 1.27 1.27)
+				)
+				(hide yes)
+			)
+		)
+		(property "Description" "Unpolarized capacitor"
+			(at 135.89 102.87 0)
+			(effects
+				(font
+					(size 1.27 1.27)
+				)
+				(hide yes)
+			)
+		)
+		(pin "2"
+		)
+		(pin "1"
+		)
+		(instances
+			(project ""
+				(path "/cfa4a98a-fd35-4db5-8ff8-6d1775bad148"
+					(reference "C1")
+					(unit 1)
+				)
